File: PLC-Hardware/untitled.kicad_sch (KiCad schematic)
At the start: 52 parts, among them J3 Conn_01x04_Pin, J4 Conn_01x04_Pin, J5 Conn_01x04_Pin, J6 Conn_01x04_Pin, U1 PC817, U17 ULN2803A, U18 ULN2803A

Commit message: Add PDF Prints
Parts:
- renumbered R1 to R32, R1 to R33, R1 to R34, R1 to R35, R5 to R36, R5 to R37, R5 to R38, R5 to R39, R1 to R40, R1 to R41, R1 to R42, R1 to R43, R5 to R44, R5 to R45, R5 to R46, R5 to R47, R1 to R48, R1 to R49, R5 to R50, R5 to R51, U1 to U19, U1 to U20, U1 to U21, U1 to U22, U1 to U23, U1 to U24, U1 to U25, U1 to U26, U1 to U27, U1 to U28
