File: Digital Logic Clock/HoursCount.kicad_sch (KiCad schematic)
At the start: 19 parts, among them U1 4081

Commit message: Clock Project
Other:
- company: (none) -> Akbar Q
- title: (none) -> Hours Counter
