File: Digital Logic Clock/MinutesCount.kicad_sch (KiCad schematic)
At the start: 19 parts, among them U1 4081

Commit message: Clock Project
Other:
- company: (none) -> Akbar Q
- title: (none) -> Minutes Counter
