File: Digital Logic Clock/SecondsCount.kicad_sch (KiCad schematic)
At the start: 19 parts, among them U1 4081

Commit message: Revise Comments
Other:
- company: (none) -> Akbar Q
- title: (none) -> Seconds Counter
Changed lines of the file:
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@@
 	(generator_version "9.0")
 	(paper "A4")
+	(title_block
+		(title "Seconds Counter")
+		(date "2023-12-24")
+		(rev "1.0")
+		(company "Akbar Q")
+	)
 	(text "Seconds Count - 59"
 		(exclude_from_sim no)
