File: Digital Logic Clock/clock-circuit.kicad_sch (KiCad schematic)
At the start: 6 parts, among them U2 NE555P

Commit message: Revise Comments
Other:
- company: (none) -> Akbar Q
- title: (none) -> Clock Signal Generator
- moved on the sheet: Cd1, Ctime1, Ra1, RaTune1, Rb1, U2
