File: NiMH Battery Charger/020 NiMH Battery Charger.kicad_sch (KiCad schematic)
At the start: 85 parts, among them J1 USB_C_Receptacle_PowerOnly_6P, U1 AMS1117-3.3, U2 ESP32-WROOM-32D, U3 AMS1117-3.3, U4 D168K

Commit message: Update to 9.0
Parts:
- renumbered D1 to D21, D1 to D22, D1 to D23, D1 to D24, D1 to D25
