File: MPPT Controller/MPPT-Controller/untitled.kicad_sch (KiCad schematic)
At the start: 29 parts, among them J5 USB_C_Receptacle_USB2.0_16P, U2 ESP32-WROOM-32D, U3 CH340C

Commit message: Add footprints partial
Parts:
- BOOT1, RESET1: footprint CustomLibrary:SwitchCustom -> Button_Switch_SMD:SW_Push_1P1T_XKB_TS-1187A
Changed lines of the file:
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@@
 			)
 		)
-		(property "Footprint" "CustomLibrary:SwitchCustom"
+		(property "Footprint" "Button_Switch_SMD:SW_Push_1P1T_XKB_TS-1187A"
 			(at 101.6 44.45 0)
 			(effects
@@
 			)
 		)
-		(property "Footprint" "CustomLibrary:SwitchCustom"
+		(property "Footprint" "Button_Switch_SMD:SW_Push_1P1T_XKB_TS-1187A"
 			(at 73.66 44.45 0)
 			(effects

Commit message: Apply Footprints
Parts:
- R13, R14, R15, R6: footprint (none) -> Resistor_SMD:R_0603_1608Metric_Pad0.98x0.95mm_HandSolder
Changed lines of the file:
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@@
 			)
 		)
-		(property "Footprint" ""
+		(property "Footprint" "Resistor_SMD:R_0603_1608Metric_Pad0.98x0.95mm_HandSolder"
 			(at 134.112 106.68 90)
 			(effects
@@
 			)
 		)
-		(property "Footprint" ""
+		(property "Footprint" "Resistor_SMD:R_0603_1608Metric_Pad0.98x0.95mm_HandSolder"
 			(at 134.112 123.19 90)
 			(effects
@@
 			)
 		)
-		(property "Footprint" ""
+		(property "Footprint" "Resistor_SMD:R_0603_1608Metric_Pad0.98x0.95mm_HandSolder"
 			(at 155.702 106.68 90)
 			(effects
@@
 			)
 		)
-		(property "Footprint" ""
+		(property "Footprint" "Resistor_SMD:R_0603_1608Metric_Pad0.98x0.95mm_HandSolder"
 			(at 155.702 123.19 90)
 			(effects
