File: MPPT Controller/MPPT-Controller/_autosave-MPPT-Controller.kicad_pcb (KiCad board)
At the start: 4 copper layers, 79 parts, among them J1 Conn_01x02_Pin, J2 Conn_01x02_Pin, J3 Conn_01x02_Pin, J4 Conn_01x02_Pin, J5 USB_C_Receptacle_USB2.0_16P, J6 Conn_01x02_Pin, Q1 IRL540N, SW1 SW_SPDT, U1 ADS1115IDGS, U2 ESP32-WROOM-32D, U3 CH340C, U4 LM1117DT-3.3, U5 LM2596S-ADJ, U6 TC4422, U7 ADS1115IDGS

Commit message: Layout
Parts:
- added HS1: Heatsink_Pad, Heatsink:Heatsink_AAVID_576802B03900G, B.Cu at (68.6, 100.5)
- added M1: Fan_4pin, Connector:FanPinHeader_1x04_P2.54mm_Vertical, F.Cu at (122.9, 81.0)
- Q1: moved to B.Cu
- moved R25 136.5 mm to (76.2, 135.9)
- moved L2 50.6 mm to (77.5, 114.3)
- moved C16 14.8 mm to (101.6, 121.9)
- moved LR3 14.8 mm to (106.4, 117.3)
- moved LR4 14.8 mm to (119.1, 117.3)
- moved J2 14.8 mm to (133.1, 119.9)
- moved C17 14.6 mm to (66.0, 121.9)
- moved U6 10.5 mm to (58.2, 64.2)
- moved Q1 8.60 mm to (71.1, 105.4)
- moved LR2 6.71 mm to (57.1, 119.0), turned to -90 degrees
- moved LR1 1.27 mm to (57.1, 106.7)
Connections:
- R1 pad 1: GND -> Net-(U5-FB)
- R1 pad 2: Net-(U5-FB) -> GND
Routing:
- added copper zone on F.Cu, net Net-(J1-Pin_2)
