File: MPPT Controller/MPPT-Controller/MPPT-Controller.kicad_sch (KiCad schematic)
At the start: 60 parts, among them J1 Conn_01x02_Pin, J2 Conn_01x02_Pin, J3 Conn_01x02_Pin, J4 Conn_01x02_Pin, J6 Conn_01x02_Pin, J7 Conn_01x02_Pin, J8 Conn_01x02_Pin, M1 Fan_4pin, Q1 IRL540N, SW1 SW_SPDT, U1 ADS1115IDGS, U4 LM1117DT-3.3, U5 LM2596S-ADJ, U6 TC4422, U7 ADS1115IDGS

Commit message: Diode
Connections:
- net +3V3: now also R29.1; no longer J8.1 (Pin_1)
- net Aux2: now also J8.1 (Pin_1), R29.2; no longer J8.2 (Pin_2), R29.1
- net GND: now also J8.2 (Pin_2); no longer R29.2
- net RDY2: now reaches U7.2 (ALERT/RDY)
- net RDY1: now reaches U1.2 (ALERT/RDY)
Other:
- moved on the sheet: J7, J8, R28, R29
