File: MPPT Controller/_autosave-MPPT-Controller.kicad_pcb (KiCad board)
At the start: 4 copper layers, 92 parts, among them J1 Conn_01x02_Pin, J2 Conn_01x02_Pin, J3 Conn_01x02_Pin, J4 Conn_01x02_Pin, J5 USB_C_Receptacle_USB2.0_16P, J6 Conn_01x02_Pin, J7 Conn_01x02_Pin, J8 Conn_01x02_Pin, J9 Conn_01x02_Pin, M1 Fan_4pin, Q1 IRL540N, SW1 SW_SPDT, U1 ADS1115IDGS, U2 ESP32-WROOM-32D, U3 CH340C, U4 LM1117DT-3.3, U5 LM2596S-ADJ, U6 TC4422, U7 ADS1115IDGS

Commit message: Save
Parts:
- moved J9 4.70 mm to (47.0, 90.9)
- moved R30 3.56 mm to (43.3, 88.9)
- moved R31 3.56 mm to (43.3, 90.4)
Routing:
- net HeatsinkT: track 0.00 -> 16.4 mm
- net SDA: track 42.9 -> 47.0 mm
- net SCL: track 42.6 -> 45.8 mm
Changed lines of the file:
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@@
 	(footprint "Resistor_SMD:R_0603_1608Metric_Pad0.98x0.95mm_HandSolder"
 		(layer "F.Cu")
-		(at 46.8395 88.9 180)
+		(at 43.2835 88.9 180)
 		(descr "Resistor SMD 0603 (1608 Metric), square (rectangular) end terminal, IPC-7351 nominal with elongated pad for handsoldering. (Body size source: IPC-SM-782 page 72, https://www.pcb-3d.com/wordpress/wp-content/uploads/ipc-sm-782a_amendment_1_and_2.pdf), generated with kicad-footprint-generator")
 		(tags "resistor handsolder")
@@
 	(footprint "Resistor_SMD:R_0603_1608Metric_Pad0.98x0.95mm_HandSolder"
 		(layer "F.Cu")
-		(at 46.8395 90.424 180)
+		(at 43.2835 90.424 180)
 		(descr "Resistor SMD 0603 (1608 Metric), square (rectangular) end terminal, IPC-7351 nominal with elongated pad for handsoldering. (Body size source: IPC-SM-782 page 72, https://www.pcb-3d.com/wordpress/wp-content/uploads/ipc-sm-782a_amendment_1_and_2.pdf), generated with kicad-footprint-generator")
 		(tags "resistor handsolder")
@@
 	(footprint "Connector_PinHeader_2.54mm:PinHeader_1x02_P2.54mm_Vertical"
 		(layer "F.Cu")
-		(at 42.291 91.059 180)
+		(at 46.99 90.937 180)
 		(descr "Through hole straight pin header, 1x02, 2.54mm pitch, single row")
 		(tags "Through hole pin header THT 1x02 2.54mm single row")
@@
 	)
 	(segment
-		(start 50.102 88.9)
-		(end 50.705 88.297)
+		(start 50.705 82.328)
+		(end 50.705 87.512)
 		(width 0.25)
 		(layer "F.Cu")
@@
 	)
 	(segment
-		(start 50.705 82.328)
-		(end 50.705 87.512)
+		(start 49.657 81.28)
+		(end 50.705 82.328)
 		(width 0.25)
 		(layer "F.Cu")
@@
 	)
 	(segment
-		(start 49.657 81.28)
-		(end 50.705 82.328)
+		(start 50.705 87.512)
+		(end 50.705 88.297)
 		(width 0.25)
 		(layer "F.Cu")
@@
 	)
 	(segment
-		(start 34.32 80.996)
-		(end 34.32 64.91)
-		(width 0.6)
+		(start 50.605 88.397)
+		(end 46.99 88.397)
+		(width 0.25)
+		(layer "F.Cu")
+		(net 51)
+	)
+	(segment
+		(start 46.487 88.9)
+		(end 46.99 88.397)
+		(width 0.8)
 		(layer "F.Cu")
 		(net 51)
@@
 	(segment
 		(start 50.705 88.297)
-		(end 50.705 87.512)
+		(end 50.605 88.397)
 		(width 0.25)
 		(layer "F.Cu")
@@
 	)
 	(segment
-		(start 47.3945 88.9)
-		(end 50.102 88.9)
-		(width 0.25)
+		(start 34.32 80.996)
+		(end 34.32 64.91)
+		(width 0.6)
+		(layer "F.Cu")
+		(net 51)
+	)
+	(segment
+		(start 44.196 88.9)
+		(end 46.487 88.9)
+		(width 0.8)
 		(layer "F.Cu")
 		(net 51)
@@
 	)
 	(segment
+		(start 51.205 88.876)
+		(end 51.205 87.512)
+		(width 0.25)
+		(layer "F.Cu")
+		(net 52)
+	)
+	(segment
 		(start 36.576 71.12)
 		(end 38.13 69.566)
@@
 	)
 	(segment
-		(start 51.205 88.43481)
-		(end 51.205 87.512)
+		(start 47.239 90.937)
+		(end 49.144 90.937)
 		(width 0.25)
 		(layer "F.Cu")
@@
 	)
 	(segment
+		(start 46.99 90.81)
+		(end 46.604 90.424)
+		(width 0.25)
+		(layer "F.Cu")
+		(net 52)
+	)
+	(segment
+		(start 44.196 90.424)
+		(end 46.477 90.424)
+		(width 0.8)
+		(layer "F.Cu")
+		(net 52)
+	)
+	(segment
 		(start 50.165 80.518)
 		(end 51.205 81.558)
@@
 	)
 	(segment
-		(start 49.21581 90.424)
-		(end 51.205 88.43481)
+		(start 49.144 90.937)
+		(end 51.205 88.876)
 		(width 0.25)
 		(layer "F.Cu")
@@
 	)
 	(segment
-		(start 51.205 81.558)
-		(end 51.205 85.598)
-		(width 0.25)
+		(start 46.477 90.424)
+		(end 46.99 90.937)
+		(width 0.8)
 		(layer "F.Cu")
 		(net 52)
 	)
 	(segment
-		(start 47.3945 90.424)
-		(end 49.21581 90.424)
+		(start 51.205 81.558)
+		(end 51.205 85.598)
 		(width 0.25)
 		(layer "F.Cu")
@@
 	)
 	(segment
+		(start 38.13 91.084)
+		(end 38.13 82.41)
+		(width 0.8)
+		(layer "F.Cu")
+		(net 85)
+	)
+	(segment
+		(start 43.566 96.52)
+		(end 38.13 91.084)
+		(width 0.8)
+		(layer "F.Cu")
+		(net 85)
+	)
+	(segment
