File: MPPT Controller/_autosave-MPPT-Controller.kicad_pcb (KiCad board)
At the start: 4 copper layers, 99 x 99 mm, 99 parts, among them J1 Conn_01x02_Pin, J10 Conn_01x02_Pin, J11 Conn_01x02_Pin, J2 Conn_01x02_Pin, J3 Conn_01x02_Pin, J4 Conn_01x02_Pin, J5 USB_C_Receptacle_USB2.0_16P, J6 Conn_01x02_Pin, J7 Conn_01x02_Pin, J8 Conn_01x02_Pin, J9 Conn_01x02_Pin, M1 Fan_4pin, Q1 IRL540N, SW1 SW_SPDT, U1 ADS1115IDGS, U2 ESP32-WROOM-32D, U3 CH340C, U4 LM1117DT-3.3, U5 LM2596S-ADJ, U6 TC4422, U7 ADS1115IDGS

Commit message: Silkscreen Layout
Parts:
- added G***: LOGO, LOGO, F.Cu at (97.0, 121.4)
- added G***: LOGO, LOGO, B.Cu at (57.1, 88.9)
- moved R26 0.32 mm to (132.2, 47.0)
Other:
- board text added: "ADC1 A3 GND Pup"
- board text added: "ADC2 A3 Pdwn 3V3"
- board text added: "ADS1115 ADC1 A1 A2"
- board text added: "ADS1115 ADC2 A1 A2"
- board text added: "AIO MMPT Development Platform - V0.1 6/25"
- board text added: "GPIO33 Pdwn 3V3"
- board text added: "Volt In 200kR/1kR ADC1 A2"
- board text added: "Volt Out 200kR/1kR ADC2 A2"
- board text removed: "ADS1115 Measure"
- board text removed: "AIO MMPT Development Platform - V1.0 6/25"
