File: MPPT Controller/MPPT-Controller.kicad_sch (KiCad schematic)
At the start: 60 parts, among them J1 Conn_01x02_Pin, J2 Conn_01x02_Pin, J3 Conn_01x02_Pin, J4 Conn_01x02_Pin, J6 Conn_01x02_Pin, J7 Conn_01x02_Pin, J8 Conn_01x02_Pin, M1 Fan_4pin, Q1 IRL540N, SW1 SW_SPDT, U1 ADS1115IDGS, U4 LM1117DT-3.3, U5 LM2596S-ADJ, U6 TC4422, U7 ADS1115IDGS

Commit message: usb c
Parts:
- added J10: Conn_01x02_Pin, TerminalBlock:TerminalBlock_Altech_AK300-2_P5.00mm, symbol Connector:Conn_01x02_Pin
- added R32, R33: 50R, Resistor_SMD:R_0603_1608Metric_Pad0.98x0.95mm_HandSolder, symbol Device:R
Connections:
- net OdiffA: now also R32.2
- net OdiffB: now also R33.2
- new net: J10.1 (Pin_1), R32.1
- new net: J10.2 (Pin_2), R33.1
Other:
- moved on the sheet: J6

Commit message: Changes
Connections:
- net GND: now also J4.1 (Pin_1); no longer J4.2 (Pin_2)
- net Vaux: now also J4.2 (Pin_2); no longer J4.1 (Pin_1)
Changed lines of the file:
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@@
 	(wire
 		(pts
-			(xy 25.4 118.11) (xy 27.94 118.11)
-		)
-		(stroke
-			(width 0)
-			(type default)
-		)
-	)
-	(wire
-		(pts
 			(xy 55.88 22.86) (xy 55.88 31.75)
 		)
@@
 	(wire
 		(pts
+			(xy 25.4 118.11) (xy 27.94 118.11)
+		)
+		(stroke
+			(width 0)
+			(type default)
+		)
+	)
+	(wire
+		(pts
 			(xy 25.4 90.17) (xy 27.94 90.17)
 		)
@@
 	(symbol
 		(lib_id "Connector:Conn_01x02_Pin")
-		(at 20.32 118.11 0)
+		(at 20.32 120.65 0)
+		(mirror x)
 		(unit 1)
 		(exclude_from_sim no)
@@
 		)
 		(property "Value" "Conn_01x02_Pin"
-			(at 27.94 122.682 0)
+			(at 27.94 116.078 0)
 			(effects
 				(font
@@
 		)
 		(property "Footprint" "TerminalBlock:TerminalBlock_Altech_AK300-2_P5.00mm"
-			(at 20.32 118.11 0)
+			(at 20.32 120.65 0)
 			(effects
 				(font
@@
 		)
 		(property "Datasheet" "~"
-			(at 20.32 118.11 0)
+			(at 20.32 120.65 0)
 			(effects
 				(font
@@
 		)
 		(property "Description" "Generic connector, single row, 01x02, script generated"
-			(at 20.32 118.11 0)
+			(at 20.32 120.65 0)
 			(effects
 				(font
