File: MPPT Controller/MPPT-Controller.kicad_pcb (KiCad board)
At the start: 4 copper layers, 92 parts, among them J1 Conn_01x02_Pin, J2 Conn_01x02_Pin, J3 Conn_01x02_Pin, J4 Conn_01x02_Pin, J5 USB_C_Receptacle_USB2.0_16P, J6 Conn_01x02_Pin, J7 Conn_01x02_Pin, J8 Conn_01x02_Pin, J9 Conn_01x02_Pin, M1 Fan_4pin, Q1 IRL540N, SW1 SW_SPDT, U1 ADS1115IDGS, U2 ESP32-WROOM-32D, U3 CH340C, U4 LM1117DT-3.3, U5 LM2596S-ADJ, U6 TC4422, U7 ADS1115IDGS

Commit message: Fix Label Name
Parts:
- moved BOOT1 37.6 mm to (64.8, 67.3)
- moved RESET1 17.3 mm to (64.8, 76.2)
- moved R7 12.7 mm to (105.4, 97.8), turned to 90 degrees
- moved C5 12.0 mm to (103.6, 97.8), turned to 90 degrees
- moved R8 7.10 mm to (109.2, 97.8), turned to 90 degrees
- moved J9 4.70 mm to (47.0, 90.9)
- moved U7 4.20 mm to (106.7, 89.7), turned to 90 degrees
- moved C6 3.84 mm to (111.0, 97.8), turned to 90 degrees
- moved R30 3.56 mm to (43.3, 88.9)
- moved R31 3.56 mm to (43.3, 90.4)
Connections:
- U7 pad 4: IdiffA -> OdiffA
- U7 pad 5: IdiffB -> OdiffB
- U7 pad 6: VoltIn -> VoltOut
Routing:
- net PWM: track 0.00 -> 76.0 mm, vias 0 -> 2
- net RST: track 0.00 -> 43.9 mm, vias 0 -> 2
- net BOOT: track 0.00 -> 27.6 mm
- net HeatsinkT: track 0.00 -> 16.4 mm
- net SDA: track 42.9 -> 47.0 mm
- net SCL: track 42.6 -> 45.8 mm

Commit message: usb c
Parts:
- added J10: Conn_01x02_Pin, TerminalBlock:TerminalBlock_Altech_AK300-2_P5.00mm, F.Cu at (219.2, 29.9)
- added R32: 50R, Resistor_SMD:R_0603_1608Metric_Pad0.98x0.95mm_HandSolder, F.Cu at (230.2, 24.2)
- added R33: 50R, Resistor_SMD:R_0603_1608Metric_Pad0.98x0.95mm_HandSolder, F.Cu at (230.2, 26.7)
- C11, C12, R27, U4: moved to B.Cu
- moved C8 231.6 mm to (49.0, 48.0), turned to -90 degrees
- moved C7 227.1 mm to (53.8, 48.0), turned to 90 degrees
- moved C12 148.3 mm to (67.1, 72.4), turned to 90 degrees
- moved C11 143.5 mm to (67.3, 76.8), turned to -90 degrees
- moved U4 119.7 mm to (59.7, 73.7), turned to 180 degrees
- moved R27 76.6 mm to (39.9, 96.5), turned to 180 degrees
- moved R26 61.2 mm to (119.6, 87.1), turned to 180 degrees
- moved TH1 55.0 mm to (125.1, 87.1), turned to 180 degrees
- moved J7 55.0 mm to (125.1, 80.0), turned to -90 degrees
- moved R28 49.0 mm to (117.5, 80.0), turned to 180 degrees
- moved R29 47.3 mm to (124.0, 74.8), turned to 180 degrees
- moved J8 44.6 mm to (118.1, 74.9), turned to -90 degrees
- moved C4 35.0 mm to (194.3, 39.8), turned to -90 degrees
- moved C3 31.6 mm to (196.8, 39.8), turned to -90 degrees
- moved R16 18.9 mm to (55.6, 56.6)
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Connections:
- U2 pad 13: unconnected-(U2-IO14-Pad13) -> Tacho
- U2 pad 16: unconnected-(U2-IO13-Pad16) -> FanPWM
Routing:
- net Net-(D1-A): track 0.00 -> 14.1 mm
- net Net-(D3-A): track 0.00 -> 13.5 mm
- net Net-(D5-A): track 0.00 -> 11.5 mm
- net Net-(D4-A): track 0.00 -> 10.3 mm
- net Net-(D2-A): track 0.00 -> 8.78 mm
- net +3V3: track 0.00 -> 4.33 mm, vias 0 -> 3
- net HeatsinkT: track 16.4 -> 19.0 mm
- net AmbientT: track 0.00 -> 2.55 mm

Commit message: Changes
Parts:
- C3, C4: moved to B.Cu
- moved C10 248.4 mm to (32.3, 53.8), turned to 90 degrees
- moved C9 242.8 mm to (39.1, 62.5)
- moved FLASH1 219.7 mm to (40.1, 47.7), turned to -90 degrees
- moved C4 78.8 mm to (118.1, 60.0), turned to 90 degrees
- moved J4 77.9 mm to (121.9, 57.2), turned to -90 degrees
- moved C3 73.9 mm to (125.7, 60.0), turned to 90 degrees
- moved R1 52.5 mm to (88.4, 63.2)
- moved C13 52.5 mm to (88.6, 65.5)
- moved C14 52.5 mm to (98.6, 59.2)
- moved C15 52.5 mm to (79.8, 74.9)
- moved D8 52.5 mm to (95.4, 79.4)
- moved L1 52.5 mm to (93.4, 71.1)
- moved R21 52.5 mm to (86.4, 74.7)
- moved R22 52.5 mm to (86.4, 71.8)
- moved U5 52.5 mm to (91.3, 54.0)
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Connections:
- FLASH1 pad 4: RST -> Rx
- FLASH1 pad 5: Tx -> RST
- FLASH1 pad 6: Rx -> Tx
- J4 pad 1: Vaux -> GND
- J4 pad 2: GND -> Vaux
Routing:
- net Tx: track 5.33 -> 15.5 mm, vias 0 -> 1
- net Rx: track 5.33 -> 14.9 mm, vias 0 -> 1
- net Net-(U3-V3): track 0.00 -> 2.87 mm

Commit message: Connectors
Parts:
- moved R6 87.8 mm to (192.0, 39.9)
- moved R14 87.7 mm to (192.0, 42.7)
- moved R15 84.2 mm to (195.6, 42.7)
- moved R13 84.1 mm to (195.6, 39.9)
- moved R32 43.9 mm to (192.0, 45.7), turned to 180 degrees
- moved R33 39.5 mm to (195.6, 45.7)
Changed lines of the file:
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@@
 	(footprint "Resistor_SMD:R_0603_1608Metric_Pad0.98x0.95mm_HandSolder"
 		(layer "F.Cu")
-		(at 279.68 42.005)
+		(at 195.58 39.878)
 		(descr "Resistor SMD 0603 (1608 Metric), square (rectangular) end terminal, IPC-7351 nominal with elongated pad for handsoldering. (Body size source: IPC-SM-782 page 72, https://www.pcb-3d.com/wordpress/wp-content/uploads/ipc-sm-782a_amendment_1_and_2.pdf), generated with kicad-footprint-generator")
 		(tags "resistor handsolder")
@@
 	(footprint "Resistor_SMD:R_0603_1608Metric_Pad0.98x0.95mm_HandSolder"
 		(layer "F.Cu")
-		(at 279.68 34.475)
+		(at 192.024 39.878)
 		(descr "Resistor SMD 0603 (1608 Metric), square (rectangular) end terminal, IPC-7351 nominal with elongated pad for handsoldering. (Body size source: IPC-SM-782 page 72, https://www.pcb-3d.com/wordpress/wp-content/uploads/ipc-sm-782a_amendment_1_and_2.pdf), generated with kicad-footprint-generator")
 		(tags "resistor handsolder")
@@
 	(footprint "Resistor_SMD:R_0603_1608Metric_Pad0.98x0.95mm_HandSolder"
 		(layer "F.Cu")
-		(at 230.2275 26.67)
+		(at 195.58 45.72)
 		(descr "Resistor SMD 0603 (1608 Metric), square (rectangular) end terminal, IPC-7351 nominal with elongated pad for handsoldering. (Body size source: IPC-SM-782 page 72, https://www.pcb-3d.com/wordpress/wp-content/uploads/ipc-sm-782a_amendment_1_and_2.pdf), generated with kicad-footprint-generator")
 		(tags "resistor handsolder")
@@
 	(footprint "Resistor_SMD:R_0603_1608Metric_Pad0.98x0.95mm_HandSolder"
 		(layer "F.Cu")
-		(at 279.68 47.025)
+		(at 195.58 42.672)
 		(descr "Resistor SMD 0603 (1608 Metric), square (rectangular) end terminal, IPC-7351 nominal with elongated pad for handsoldering. (Body size source: IPC-SM-782 page 72, https://www.pcb-3d.com/wordpress/wp-content/uploads/ipc-sm-782a_amendment_1_and_2.pdf), generated with kicad-footprint-generator")
 		(tags "resistor handsolder")
@@
 	(footprint "Resistor_SMD:R_0603_1608Metric_Pad0.98x0.95mm_HandSolder"
 		(layer "F.Cu")
-		(at 279.68 44.515)
+		(at 192.024 42.672)
 		(descr "Resistor SMD 0603 (1608 Metric), square (rectangular) end terminal, IPC-7351 nominal with elongated pad for handsoldering. (Body size source: IPC-SM-782 page 72, https://www.pcb-3d.com/wordpress/wp-content/uploads/ipc-sm-782a_amendment_1_and_2.pdf), generated with kicad-footprint-generator")
 		(tags "resistor handsolder")
@@
 	(footprint "Resistor_SMD:R_0603_1608Metric_Pad0.98x0.95mm_HandSolder"
 		(layer "F.Cu")
-		(at 230.2275 24.16)
+		(at 192.024 45.72 180)
 		(descr "Resistor SMD 0603 (1608 Metric), square (rectangular) end terminal, IPC-7351 nominal with elongated pad for handsoldering. (Body size source: IPC-SM-782 page 72, https://www.pcb-3d.com/wordpress/wp-content/uploads/ipc-sm-782a_amendment_1_and_2.pdf), generated with kicad-footprint-generator")
 		(tags "resistor handsolder")
 		(property "Reference" "R32"
-			(at 0 -1.43 0)
+			(at 0 1.397 0)
 			(layer "F.SilkS")
 			(effects
@@
 		(attr smd)
 		(fp_line
-			(start -0.254724 -0.5225)
-			(end 0.254724 -0.5225)
+			(start -0.254724 0.5225)
+			(end 0.254724 0.5225)
 			(stroke
 				(width 0.12)
@@
 		)
 		(fp_line
-			(start -0.254724 0.5225)
-			(end 0.254724 0.5225)
+			(start -0.254724 -0.5225)
+			(end 0.254724 -0.5225)
 			(stroke
 				(width 0.12)
@@
 		)
 		(fp_line
-			(start -1.65 -0.73)
-			(end 1.65 -0.73)
+			(start 1.65 0.73)
+			(end -1.65 0.73)
 			(stroke
 				(width 0.05)
@@
 		)
 		(fp_line
-			(start -1.65 0.73)
-			(end -1.65 -0.73)
+			(start 1.65 -0.73)
+			(end 1.65 0.73)
 			(stroke
 				(width 0.05)
@@
 		)
 		(fp_line
-			(start 1.65 -0.73)
-			(end 1.65 0.73)
+			(start -1.65 0.73)
+			(end -1.65 -0.73)
 			(stroke
 				(width 0.05)
@@
 		)
 		(fp_line
-			(start 1.65 0.73)
-			(end -1.65 0.73)
+			(start -1.65 -0.73)
+			(end 1.65 -0.73)
 			(stroke
 				(width 0.05)
@@
 		)
 		(fp_line
-			(start -0.8 -0.4125)
-			(end 0.8 -0.4125)
+			(start 0.8 0.4125)
+			(end -0.8 0.4125)
 			(stroke
 				(width 0.1)
@@
 		)
 		(fp_line
-			(start -0.8 0.4125)
-			(end -0.8 -0.4125)
+			(start 0.8 -0.4125)
+			(end 0.8 0.4125)
 			(stroke
 				(width 0.1)
@@
 		)
 		(fp_line
-			(start 0.8 -0.4125)
-			(end 0.8 0.4125)
+			(start -0.8 0.4125)
+			(end -0.8 -0.4125)
 			(stroke
 				(width 0.1)
@@
 		)
 		(fp_line
-			(start 0.8 0.4125)
-			(end -0.8 0.4125)
+			(start -0.8 -0.4125)
+			(end 0.8 -0.4125)
 			(stroke
 				(width 0.1)
@@
 		)
 		(pad "1" smd roundrect
-			(at -0.9125 0)
+			(at -0.9125 0 180)
 			(size 0.975 0.95)
 			(layers "F.Cu" "F.Mask" "F.Paste")
@@
 		)
 		(pad "2" smd roundrect
-			(at 0.9125 0)
+			(at 0.9125 0 180)
 			(size 0.975 0.95)
 			(layers "F.Cu" "F.Mask" "F.Paste")

Commit message: Connector Layout
Parts:
- moved R13 155.4 mm to (50.0, 94.2)
- moved R6 154.7 mm to (47.5, 95.1), turned to 90 degrees
- moved J10 105.6 mm to (121.9, 71.1), turned to -90 degrees
- moved J6 100.6 mm to (121.9, 83.6), turned to -90 degrees
- moved R15 96.5 mm to (114.3, 94.7), turned to 90 degrees
- moved R14 95.6 mm to (114.3, 98.3), turned to 90 degrees
- moved R33 75.4 mm to (122.3, 63.5)
- moved R32 75.4 mm to (118.7, 63.5)
- moved R26 36.8 mm to (155.8, 80.6)
- moved J7 36.8 mm to (161.3, 76.1)
- moved R28 36.8 mm to (153.7, 76.1)
- moved TH1 36.8 mm to (161.3, 80.7)
- moved J8 36.1 mm to (153.7, 71.1)
- moved R29 36.1 mm to (159.6, 71.0)
- moved SW1 35.6 mm to (125.7, 33.0)
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Routing:
- net VoltIn: track 0.00 -> 9.83 mm
- net Aux1: track 0.00 -> 7.96 mm, vias 0 -> 1
- net Vin: track 0.00 -> 3.13 mm
- net GND: track 0.00 -> 2.73 mm, vias 63 -> 64
- net +3V3: track 4.33 -> 5.76 mm, vias 3 -> 4

Commit message: Shunt Tap
Parts:
- moved J3 152.8 mm to (36.8, 122.1), turned to 90 degrees
- moved R5 143.8 mm to (39.9, 111.3), turned to 90 degrees
- moved R4 142.5 mm to (41.9, 111.3), turned to 90 degrees
- moved R33 16.3 mm to (112.1, 76.2), turned to 180 degrees
- moved J1 10.2 mm to (36.8, 134.6)
- moved R32 10.1 mm to (112.1, 71.1)
Routing:
- net IdiffB: track 5.05 -> 32.8 mm, vias 0 -> 2
- net IdiffA: track 4.83 -> 30.6 mm, vias 0 -> 2
- net Net-(J3-Pin_1): track 0.00 -> 13.1 mm
- net Net-(J3-Pin_2): track 0.00 -> 7.55 mm

Commit message: Layout Changes
Parts:
- D9: moved to B.Cu
- SW1: moved to F.Cu
- moved R11 183.3 mm to (58.7, 78.7), turned to 180 degrees
- moved R12 183.2 mm to (58.4, 68.6), turned to 180 degrees
- moved D9 175.6 mm to (43.9, 49.4), turned to 90 degrees
- moved R26 39.0 mm to (120.3, 64.7)
- moved TH1 39.0 mm to (125.7, 64.8)
- moved J7 38.6 mm to (125.7, 61.0)
- moved R28 38.6 mm to (118.1, 61.0)
- moved J8 38.2 mm to (118.1, 57.3)
- moved R29 38.2 mm to (124.0, 57.1)
- moved SW1 18.9 mm to (113.0, 47.0), turned to 0 degrees
- moved F2 0.77 mm to (109.2, 63.5)
- moved R7 0.57 mm to (105.7, 98.3)
- moved C5 0.57 mm to (103.9, 98.3)
- turned C7 to -90 degrees
Routing:
- net Net-(J5-SHIELD): track 0.00 -> 21.4 mm
- net RST: track 43.9 -> 52.6 mm
- net OdiffB: track 0.00 -> 6.21 mm
- net OdiffA: track 0.00 -> 6.21 mm
- net +3V3: track 5.76 -> 10.2 mm, vias 4 -> 6
- net Vaux: track 0.00 -> 3.67 mm, vias 0 -> 2
- net Net-(D9-A): track 2.70 -> 4.65 mm, vias 0 -> 1
- net BOOT: track 27.6 -> 29.2 mm
- added copper zone on In2.Cu, net Net-(D9-A)
- added copper zone on F.Cu, net Net-(SW1-B)
- added copper zone on F.Cu, net Vaux
- removed copper zone on B.Cu, net Net-(SW1-B)

Commit message: Pre Verification Draft
Parts:
- moved J4 2.54 mm to (121.9, 48.3)
- moved C3 2.54 mm to (125.7, 51.1)
- moved C4 2.54 mm to (118.1, 51.1)
- moved F2 2.54 mm to (109.2, 66.0)
- moved SW1 2.54 mm to (113.0, 49.5)
- moved J7 1.78 mm to (125.7, 62.7)
- moved J8 1.78 mm to (118.1, 59.0)
- moved R28 1.78 mm to (118.1, 62.7)
- moved R29 1.78 mm to (124.0, 58.9)
- moved R26 1.52 mm to (120.3, 66.3)
- moved TH1 1.52 mm to (125.7, 66.3)
Changed lines of the file:
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@@
 	(footprint "Resistor_THT:R_Axial_DIN0204_L3.6mm_D1.6mm_P1.90mm_Vertical"
 		(layer "F.Cu")
-		(at 125.73 64.77 180)
+		(at 125.73 66.294 180)
 		(descr "Resistor, Axial_DIN0204 series, Axial, Vertical, pin pitch=1.9mm, 0.167W, length*diameter=3.6*1.6mm^2, http://cdn-reichelt.de/documents/datenblatt/B400/1_4W%23YAG.pdf")
 		(tags "Resistor Axial_DIN0204 series Axial Vertical pin pitch 1.9mm 0.167W length 3.6mm diameter 1.6mm")
 		(property "Reference" "TH1"
-			(at -2.032 0 90)
+			(at -2.032 -0.254 90)
 			(layer "F.SilkS")
 			(effects
@@
 	(footprint "LED_SMD:LED_0805_2012Metric_Pad1.15x1.40mm_HandSolder"
 		(layer "F.Cu")
-		(at 120.262 64.746 180)
+		(at 120.262 66.27 180)
 		(descr "LED SMD 0805 (2012 Metric), square (rectangular) end terminal, IPC-7351 nominal, (Body size source: https://docs.google.com/spreadsheets/d/1BsfQQcO9C6DZCsRaXUlFlo91Tg2WpOkGARC1WS5S8t0/edit?usp=sharing), generated with kicad-footprint-generator")
 		(tags "LED handsolder")
@@
 	(footprint "LED_SMD:LED_0805_2012Metric_Pad1.15x1.40mm_HandSolder"
 		(layer "F.Cu")
-		(at 118.11 60.96 180)
+		(at 118.11 62.738 180)
 		(descr "LED SMD 0805 (2012 Metric), square (rectangular) end terminal, IPC-7351 nominal, (Body size source: https://docs.google.com/spreadsheets/d/1BsfQQcO9C6DZCsRaXUlFlo91Tg2WpOkGARC1WS5S8t0/edit?usp=sharing), generated with kicad-footprint-generator")
 		(tags "LED handsolder")
@@
 	(footprint "Connector_PinHeader_2.54mm:PinHeader_1x03_P2.54mm_Vertical"
 		(layer "F.Cu")
-		(at 113.03 46.99)
+		(at 113.03 49.53)
 		(descr "Through hole straight pin header, 1x03, 2.54mm pitch, single row")
 		(tags "Through hole pin header THT 1x03 2.54mm single row")
@@
 	(footprint "LED_SMD:LED_0805_2012Metric_Pad1.15x1.40mm_HandSolder"
 		(layer "F.Cu")
-		(at 124.034 57.15 180)
+		(at 124.034 58.928 180)
 		(descr "LED SMD 0805 (2012 Metric), square (rectangular) end terminal, IPC-7351 nominal, (Body size source: https://docs.google.com/spreadsheets/d/1BsfQQcO9C6DZCsRaXUlFlo91Tg2WpOkGARC1WS5S8t0/edit?usp=sharing), generated with kicad-footprint-generator")
 		(tags "LED handsolder")
@@
 	(footprint "Connector_PinHeader_2.54mm:PinHeader_1x02_P2.54mm_Vertical"
 		(layer "F.Cu")
-		(at 118.11 57.258 -90)
+		(at 118.11 59.036 -90)
 		(descr "Through hole straight pin header, 1x02, 2.54mm pitch, single row")
 		(tags "Through hole pin header THT 1x02 2.54mm single row")
@@
 	(footprint "Connector_PinHeader_2.54mm:PinHeader_1x02_P2.54mm_Vertical"
 		(layer "F.Cu")
-		(at 125.73 60.96 -90)
+		(at 125.73 62.738 -90)
 		(descr "Through hole straight pin header, 1x02, 2.54mm pitch, single row")
 		(tags "Through hole pin header THT 1x02 2.54mm single row")
@@
 	(footprint "TerminalBlock:TerminalBlock_Altech_AK300-2_P5.00mm"
 		(layer "F.Cu")
-		(at 121.92 45.8 -90)
+		(at 121.92 48.34 -90)
 		(descr "Altech AK300 terminal block, pitch 5.0mm, 45 degree angled, see http://www.mouser.com/ds/2/16/PCBMETRC-24178.pdf")
 		(tags "Altech AK300 terminal block pitch 5.0mm")
@@
 	(footprint "Fuse:Fuseholder_Clip-5x20mm_Bel_FC-203-22_Lateral_P17.80x5.00mm_D1.17mm_Horizontal"
 		(layer "B.Cu")
-		(at 109.22 63.51 90)
+		(at 109.22 66.05 90)
 		(descr "Fuseholder Clips, 5x20mm Cylinder Fuse, Pins Lateral, Horizontal, Bel FC-203-22, https://www.belfuse.com/resources/datasheets/circuitprotection/ds-cp-0672-fuse-clips-series.pdf")
 		(tags "fuse clip open")
@@
 	(footprint "Capacitor_SMD:C_0603_1608Metric_Pad1.08x0.95mm_HandSolder"
 		(layer "B.Cu")
-		(at 125.73 48.565 90)
+		(at 125.73 51.105 90)
 		(descr "Capacitor SMD 0603 (1608 Metric), square (rectangular) end terminal, IPC-7351 nominal with elongated pad for handsoldering. (Body size source: IPC-SM-782 page 76, https://www.pcb-3d.com/wordpress/wp-content/uploads/ipc-sm-782a_amendment_1_and_2.pdf), generated with kicad-footprint-generator")
 		(tags "capacitor handsolder")
@@
 	(footprint "Capacitor_SMD:C_0603_1608Metric_Pad1.08x0.95mm_HandSolder"
 		(layer "B.Cu")
-		(at 118.11 48.565 90)
+		(at 118.11 51.105 90)
 		(descr "Capacitor SMD 0603 (1608 Metric), square (rectangular) end terminal, IPC-7351 nominal with elongated pad for handsoldering. (Body size source: IPC-SM-782 page 76, https://www.pcb-3d.com/wordpress/wp-content/uploads/ipc-sm-782a_amendment_1_and_2.pdf), generated with kicad-footprint-generator")
 		(tags "capacitor handsolder")
@@
 	)
 	(via
-		(at 125.222 51.054)
+		(at 125.222 53.594)
 		(size 1)
 		(drill 0.5)
@@
 	)
 	(via
-		(at 118.618 51.054)
+		(at 118.618 53.594)
 		(size 1)
 		(drill 0.5)
@@
 	)
 	(segment
-		(start 125.73 49.4275)
-		(end 125.73 50.546)
+		(start 125.73 51.9675)
+		(end 125.73 53.086)
 		(width 0.4)
 		(layer "B.Cu")
@@
 	)
 	(segment
-		(start 125.73 50.546)
-		(end 125.222 51.054)
+		(start 125.73 53.086)
+		(end 125.222 53.594)
 		(width 0.4)
 		(layer "B.Cu")
@@
 	)
 	(segment
-		(start 118.618 51.054)
-		(end 118.11 50.546)
+		(start 118.618 53.594)
+		(end 118.11 53.086)
 		(width 0.4)
 		(layer "B.Cu")
@@
 	)
 	(segment
-		(start 118.11 50.546)
-		(end 118.11 49.4275)
+		(start 118.11 53.086)
+		(end 118.11 51.9675)
 		(width 0.4)
 		(layer "B.Cu")
@@
 	)
 	(segment
-		(start 119.135 60.96)
-		(end 123.19 60.96)
+		(start 119.135 62.738)
+		(end 123.19 62.738)
 		(width 1.2)
 		(layer "F.Cu")
@@
 	)
 	(segment
-		(start 123.83 64.77)
-		(end 121.311 64.77)
+		(start 123.83 66.294)
+		(end 121.311 66.294)
 		(width 1.2)
 		(layer "F.Cu")
@@
 	)
 	(segment
-		(start 121.311 64.77)
-		(end 121.287 64.746)
+		(start 121.311 66.294)
+		(end 121.287 66.27)
 		(width 1.2)
 		(layer "F.Cu")
@@
 		(polygon
 			(pts
-				(xy 128.397 43.053) (xy 128.397 54.102) (xy 115.824 54.102) (xy 115.824 48.133) (xy 111.633 48.133)
-				(xy 111.633 43.053)
+				(xy 128.397 45.593) (xy 128.397 56.642) (xy 115.824 56.642) (xy 115.824 50.673) (xy 111.633 50.673)
+				(xy 111.633 45.593)
 			)
 		)
@@
 		(polygon
 			(pts
-				(xy 114.808 50.673) (xy 114.808 48.514) (xy 110.998 48.514) (xy 110.998 43.053) (xy 102.489 43.053)
-				(xy 102.489 50.673)
+				(xy 114.808 53.213) (xy 114.808 51.054) (xy 110.998 51.054) (xy 110.998 45.593) (xy 102.489 45.593)
+				(xy 102.489 53.213)
 			)
 		)
@@
 		(polygon
 			(pts
-				(xy 102.87 65.532) (xy 98.298 64.008) (xy 94.234 64.008) (xy 94.234 59.436) (xy 110.998 59.436)
-				(xy 110.998 65.532)
+				(xy 103.886 68.406) (xy 99.568 65.405) (xy 94.234 65.358) (xy 94.234 60.786) (xy 110.998 60.786)
+				(xy 110.998 68.406)
 			)
 		)
